File: PCB/Ebyte_E79.kicad_sch (KiCad schematic)
At the start: 15 parts, among them J10 JTAG, J4 ANT, SW1 BOOT, SW5 RESET, U28 ESP32-C3_OLED, U29 Ebyte_E79

Commit message: Move KiCad files to PCB
Parts:
- removed D15: SP4020, Diode_SMD:D_SOD-323, symbol Diode:5KPxxA
- removed SW5: RESET, Button_Switch_SMD:SW_Push_1P1T_NO_CK_KMR2, symbol Switch:SW_Push
- added D5: SP4020, Diode_SMD:D_SOD-323, symbol Diode:5KPxxA
- added SW3: BOOT, Button_Switch_SMD:SW_Push_1P1T_NO_CK_KMR2, symbol Switch:SW_Push
- SW1: value BOOT -> RESET
Connections:
- net BOOT: now also R2.2, D5.1 (A1), SW3.2; no longer D1.1 (A1), R1.2, SW1.2
- net GND: now also D5.2 (A2), SW3.1
- net ~{RST}: now also D1.1 (A1), R1.2, SW1.2; no longer R2.2
