File: PCB/KiCad/Ai-Thinker-Ra-09.kicad_sch (KiCad schematic)
At the start: 27 parts, among them J11 Conn_01x03_Pin, J12 USB_C_Receptacle_USB2.0_14P, J9 Conn_01x03_Pin, SW4 BOOT, SW6 RESET, U33 AMS1117-3.3, U44 RA-09, U45 CH340C

Commit message: Fix RA-09 carrier UART and BOOT routing
Parts:
- removed J11: Conn_01x03_Pin, Connector_PinHeader_2.54mm:PinHeader_1x03_P2.54mm_Vertical, symbol Connector:Conn_01x03_Pin
Connections:
- net RX1 is gone; now on net TX: U44.15 (RX1)
- net RX2 is gone; now on net TX2: U44.21 (TX2)
- net BOOT: now also U44.44 (PH3); no longer U44.45 (H3)
- net GND: now also U44.45 (GND)
- net TX: now also U44.22 (RX2)
- net TX2: no longer U44.22 (RX2)
- net at U44.1 (NC), U44.19 (NC), U44.2 (NC)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: no longer U44.44 (NC)
Changed lines of the file:
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@@
 	(wire
 		(pts
-			(xy 182.88 36.83) (xy 187.96 36.83)
-		)
-		(stroke
-			(width 0)
-			(type default)
-		)
-	)
-	(wire
-		(pts
 			(xy 114.3 45.72) (xy 106.68 45.72)
 		)
@@
 	(wire
 		(pts
-			(xy 177.8 34.29) (xy 187.96 34.29)
-		)
-		(stroke
-			(width 0)
-			(type default)
-		)
-	)
-	(wire
-		(pts
 			(xy 31.75 87.63) (xy 40.64 87.63)
 		)
@@
 	(wire
 		(pts
-			(xy 182.88 31.75) (xy 187.96 31.75)
-		)
-		(stroke
-			(width 0)
-			(type default)
-		)
-	)
-	(wire
-		(pts
 			(xy 31.75 85.09) (xy 31.75 87.63)
 		)
@@
 		)
 	)
-	(label "RX2"
-		(at 182.88 36.83 0)
-		(effects
-			(font
-				(size 1.27 1.27)
-			)
-			(justify left bottom)
-		)
-	)
 	(label "TX2"
 		(at 146.05 36.83 0)
@@
 		)
 	)
-	(label "RX1"
+	(label "TX"
 		(at 69.85 68.58 0)
 		(effects
@@
 		)
 	)
-	(label "RX2"
+	(label "TX2"
 		(at 114.3 45.72 180)
 		(effects
@@
 		)
 	)
-	(label "RX1"
-		(at 182.88 31.75 0)
-		(effects
-			(font
-				(size 1.27 1.27)
-			)
-			(justify left bottom)
-		)
-	)
 	(label "+3V3"
 		(at 134.62 171.45 180)
@@
 		)
 	)
-	(label "TX2"
+	(label "TX"
 		(at 114.3 48.26 180)
 		(effects
@@
 					(unit 1)
 				)
-			)
-		)
-	)
-	(symbol
-		(lib_id "Connector:Conn_01x03_Pin")
-		(at 193.04 34.29 0)
-		(mirror y)
-		(unit 1)
-		(body_style 1)
-		(exclude_from_sim no)
-		(in_bom yes)
-		(on_board yes)
-		(in_pos_files yes)
-		(dnp no)
-		(property "Reference" "J11"
-			(at 193.04 24.638 0)
-			(show_name no)
-			(do_not_autoplace no)
-			(effects
-				(font
-					(size 1.27 1.27)
-				)
-			)
-		)
-		(property "Value" "Conn_01x03_Pin"
-			(at 193.04 27.178 0)
-			(show_name no)
-			(do_not_autoplace no)
-			(effects
-				(font
-					(size 1.27 1.27)
-				)
-			)
-		)
-		(property "Footprint" "Connector_PinHeader_2.54mm:PinHeader_1x03_P2.54mm_Vertical"
-			(at 193.04 34.29 0)
-			(hide yes)
-			(show_name no)
-			(do_not_autoplace no)
-			(effects
-				(font
-					(size 1.27 1.27)
-				)
-			)
-		)
-		(property "Datasheet" ""
-			(at 193.04 34.29 0)
-			(hide yes)
-			(show_name no)
-			(do_not_autoplace no)
-			(effects
-				(font
-					(size 1.27 1.27)
-				)
-			)
-		)
-		(property "Description" "Generic connector, single row, 01x03, script generated"
-			(at 193.04 34.29 0)
-			(hide yes)
-			(show_name no)
-			(do_not_autoplace no)
-			(effects
-				(font
-					(size 1.27 1.27)
-				)
-			)
-		)
-		(pin "1"
-		)
-		(pin "3"
-		)
-		(pin "2"
-		)
-		(instances
-			(project "module_radio"
-				(path "/9790d703-fd6a-40c9-8b52-2dd780028164/243ab3ae-c770-4132-a7f2-2763056a5d01"
-					(reference "J11")
-					(unit 1)
-				)
