File: PCB/KiCad/module_radio.kicad_pcb (KiCad board)
At the start: 2 copper layers, 376.1 x 352.9 mm, 176 parts, among them IC2 E22-400M30S, J1 ANT, J10 JTAG, J11 Conn_01x03_Pin, J12 USB_C_Receptacle_USB2.0_14P, J13 USB_C_Receptacle_USB2.0_14P, J14 ANT, J15 JTAG, J2 ANT, J3 ANT, J4 ANT, J5 ANT, J6 ANT, J7 ANT, J8 ANT, J9 Conn_01x03_Pin, Q1 BC847, Q2 BC847, SW1 RESET, SW2 RESET, SW3 BOOT, SW4 BOOT, SW5 BOOT, SW6 RESET, U1 ESP32-C3_OLED, U10 RFM69HCW, U11 RA-02, U12 RA-01, U13 CC1101, U14 E28-2G4M12XX, U15 ESP32-C3_OLED, U16 ESP32-C3_OLED, U17 ESP32-C3_OLED, U18 ESP32-C3_OLED, U19 ESP32-C3_OLED, U2 Ai-Thinker-Ra-01, U20 ESP32-C3_OLED, U21 ESP32-C3_OLED, U22 ESP32-C3_OLED, U23 ESP32-C3_OLED, U24 ESP32-C3_OLED, U25 ESP32-C3_OLED, U26 ESP32-C3_OLED, U27 ESP32-C3_OLED, U28 ESP32-C3_OLED, U29 Ebyte_E79, U3 Ai-Thinker-Ra-02, U30 ESP32-C3_OLED, U31 TI-CC1101, U32 HC-12, U33 AMS1117-3.3, U34 ESP32-C3_OLED, U35 Ebyte_E79, U36 ESP32-C3_OLED, U37 Ebyte_E280, U38 ESP32-C3_OLED, U39 Ebyte_E79, U4 XL1276-D01, U40 ESP32-C3_OLED, U41 Ebyte_E79, U42 ESP32-C3_OLED, U43 CH9340C, U44 RA-09, U45 CH340C, U46 Ebyte_E79, U48 AMS1117-3.3, U5 NRF24L01, U6 nRF24L01+PA+LNA, U7 E32-433T20D, U8 SX127x, U9 E32-433T33D

Commit message: Fix RA-09 carrier UART and BOOT routing
Parts:
- removed J11: Conn_01x03_Pin, Connector_PinHeader_2.54mm:PinHeader_1x03_P2.54mm_Vertical
Connections:
- U44 pad 15: /Ai-Thinker-Ra-9/RX1 -> /Ai-Thinker-Ra-9/TX
- U44 pad 21: /Ai-Thinker-Ra-9/RX2 -> /Ai-Thinker-Ra-9/TX2
- U44 pad 22: /Ai-Thinker-Ra-9/TX2 -> /Ai-Thinker-Ra-9/TX
- U44 pad 44: unconnected-(U44-NC-Pad44) -> /Ai-Thinker-Ra-9/BOOT
- U44 pad 45: /Ai-Thinker-Ra-9/BOOT -> GND
Routing:
- net /Ai-Thinker-Ra-9/TX: track 18.7 -> 51.1 mm, vias 0 -> 2
- net /Ai-Thinker-Ra-9/RX2: track 22.1 -> 0.00 mm, vias 2 -> 0
- net /Ai-Thinker-Ra-9/RX1: track 20.5 -> 0.00 mm, vias 2 -> 0
- net GND: track 486.6 -> 487.8 mm
- net /Ai-Thinker-Ra-9/BOOT: track 55.7 -> 56.2 mm
Other:
- board text removed: "RX1"
- board text removed: "RX2"
